File: pcb/Shortcut_Master.kicad_pcb (KiCad board)
At the start: 2 copper layers, 78.5 x 52.9 mm, 25 parts, among them J1 Conn_01x04, SW0 SW_Push, SW1 SW_Push, SW2 SW_Push, SW3 SW_Push, SW4 SW_Push, SW5 SW_Push, SW6 RotaryEncoder_Switch, U2 XIAO-RP2040-DIP

Commit message: .
Parts:
- D1, D12, D13, D2, D3, D4: footprint LED_SMD:LED_SK6812MINI_PLCC4_3.5x3.5mm_P1.75mm -> Hackclub Footprints:MX_SK6812MINI-E_REV; moved to F.Cu
- moved D4 6.81 mm to (216.7, 127.5), turned to -90 degrees
- moved D3 6.52 mm to (216.7, 83.0), turned to -90 degrees
- moved D2 5.30 mm to (178.7, 76.0), turned to 0 degrees
- moved D13 4.90 mm to (176.2, 124.6), turned to 0 degrees
- moved D1 4.55 mm to (142.9, 83.1), turned to -90 degrees
- moved D12 4.16 mm to (142.5, 127.7), turned to -90 degrees
Routing:
- net GND: track 249.0 -> 223.6 mm, vias 1 -> 5
- net SCL: track 29.5 -> 15.9 mm
- net Net-(D3-DOUT): track 53.6 -> 40.7 mm
- net ROW0: track 71.1 -> 80.2 mm, vias 0 -> 1
- net Pin1: track 57.3 -> 50.1 mm, vias 1 -> 0
- net +5V: track 234.1 -> 228.4 mm, vias 3 -> 4
- net Pin2: track 53.1 -> 58.6 mm
- net Net-(D1-DOUT): track 40.0 -> 44.1 mm
- net COL1: track 52.1 -> 55.8 mm, vias 0 -> 1
- net Net-(D2-DOUT): track 31.0 -> 34.7 mm
- net ROW1: track 47.7 -> 51.3 mm, vias 2 -> 1
- net Net-(D9-A): track 34.2 -> 30.7 mm
- net Net-(D5-A): track 43.3 -> 40.0 mm
- net ROW2: track 54.3 -> 57.0 mm
- net Net-(D8-A): track 49.8 -> 47.5 mm
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
Commit message: new design
Parts:
- moved U2 4.34 mm to (152.5, 84.7)
- moved D1 3.35 mm to (142.7, 79.8)
- moved D2 3.35 mm to (178.5, 72.7)
- moved D3 3.35 mm to (216.5, 79.6)
- moved J1 3.35 mm to (136.4, 75.9)
- moved SW6 0.60 mm to (207.4, 90.4)
- turned SW0 to 0 degrees
- turned SW1 to 0 degrees
- turned SW2 to 0 degrees
- turned SW3 to 0 degrees
- turned SW4 to 0 degrees
- turned SW5 to 0 degrees
Routing:
- net Net-(D12-DIN): track 76.0 -> 100.6 mm
- net Net-(D6-A): track 64.8 -> 49.5 mm
- net Net-(D8-A): track 47.5 -> 34.0 mm
- net Net-(D9-A): track 30.7 -> 18.4 mm
- net COL2: track 70.7 -> 59.4 mm, vias 1 -> 2
- net Pin1: track 50.1 -> 59.2 mm
- net +5V: track 228.4 -> 220.1 mm
- net COL0: track 89.3 -> 81.3 mm, vias 1 -> 0
- net Net-(D10-A): track 30.2 -> 22.4 mm
- net ROW0: track 80.2 -> 72.4 mm, vias 1 -> 0
- net Net-(D3-DOUT): track 40.7 -> 48.4 mm
- net Pin2: track 58.6 -> 50.9 mm
- net Net-(D5-A): track 40.0 -> 32.4 mm
- net Net-(D7-A): track 25.8 -> 18.4 mm
- net Net-(D1-DOUT): track 44.1 -> 49.5 mm
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Other:
- board size 78.5 x 52.9 mm -> 78.5 x 56.5 mm
